Commit message: Auto build xacro files for models on catkin_make

File: src/robot_simulation/models/SDS_Chassis/model.xacro (robot description, xacro)
@@ -31,15 +31,4 @@
                 </mesh>
               </geometry>
-              <material>
-                <lighting>1</lighting>
-                <script>
-                  <uri>file://media/materials/scripts/gazebo.material</uri>
-                  <name>Gazebo/Grey</name>
-                </script>
-                <shader type='pixel'>
-                  <normal_map>__default__</normal_map>
-                </shader>
-                <emissive>0 0 0 1</emissive>
-              </material>
               <transparency>0</transparency>
               <cast_shadows>1</cast_shadows>

File: src/robot_simulation/models/SDS_Module/SDS_Module.xacro (robot description, xacro)
@@ -34,4 +34,90 @@
                     </mesh>
                 </geometry>
+                <transparency>0</transparency>
+                <cast_shadows>1</cast_shadows>
+            </visual>
+            <collision name='collision'>
+                <laser_retro>0</laser_retro>
+                <max_contacts>10</max_contacts>
+                <pose>0 0 0 0 -0 0</pose>
+                <geometry>
+                    <mesh>
+                        <uri>$(find robot_simulation)/models/SDS_Module/SDS_Fixed_Collision.dae</uri>
+                        <scale>1 1 1</scale>
+                    </mesh>
+                </geometry>
+                <surface>
+                    <friction>
+                        <ode>
+                            <mu>1</mu>
+                            <mu2>1</mu2>
+                            <fdir1>0 0 0</fdir1>
+                            <slip1>0</slip1>
+                            <slip2>0</slip2>
+                        </ode>
+                        <torsional>
+                            <coefficient>1</coefficient>
+                            <patch_radius>0</patch_radius>
+                            <surface_radius>0</surface_radius>
+                            <use_patch_radius>1</use_patch_radius>
+                            <ode>
+                                <slip>0</slip>
+                            </ode>
+                        </torsional>
+                    </friction>
+                    <bounce>
+                        <restitution_coefficient>0</restitution_coefficient>
+                        <threshold>1e+06</threshold>
+                    </bounce>
+                    <contact>
+                        <collide_without_contact>0</collide_without_contact>
+                        <collide_without_contact_bitmask>1</collide_without_contact_bitmask>
+                        <collide_bitmask>1</collide_bitmask>
+                        <ode>
+                            <soft_cfm>0</soft_cfm>
+                            <soft_erp>0.2</soft_erp>
+                            <kp>1e+13</kp>
+                            <kd>1</kd>
+                            <max_vel>0.01</max_vel>
+                            <min_depth>0</min_depth>
+                        </ode>
+                        <bullet>
+                            <split_impulse>1</split_impulse>
+                            <split_impulse_penetration_threshold>-0.01</split_impulse_penetration_threshold>
+                            <soft_cfm>0</soft_cfm>
+                            <soft_erp>0.2</soft_erp>
+                            <kp>1e+13</kp>
+                            <kd>1</kd>
+                        </bullet>
+                    </contact>
+                </surface>
+            </collision>
+        </link>
+        <link name='${model_name}_Rotation'>
+            <inertial>
+                <mass>0.59</mass>
+                <inertia>
+                    <ixx>0.0006558</ixx>
+                    <ixy>0</ixy>
+                    <ixz>0</ixz>
+                    <iyy>0.00065583</iyy>
+                    <iyz>0</iyz>
+                    <izz>0.00074316</izz>
+                </inertia>
+                <pose>0 0 0 0 -0 0</pose>
+            </inertial>
+            <pose>${x + 6.9e-05} ${y} ${z + 0.026037} ${roll} ${pitch} ${yaw}</pose>
+            <gravity>1</gravity>
+            <self_collide>0</self_collide>
+            <kinematic>0</kinematic>
+            <enable_wind>0</enable_wind>
+            <visual name='visual'>
+                <pose>0 0 0 0 -0 0</pose>
+                <geometry>
+                    <mesh>
+                        <uri>$(find robot_simulation)/models/SDS_Module/SDS_Rotation.dae</uri>
+                        <scale>1 1 1</scale>
+                    </mesh>
+                </geometry>
                 <material>
                     <lighting>1</lighting>
@@ -57,5 +143,5 @@
                 <geometry>
                     <mesh>
-                        <uri>$(find robot_simulation)/models/SDS_Module/SDS_Fixed_Collision.dae</uri>
+                        <uri>$(find robot_simulation)/models/SDS_Module/SDS_Rotation_Collision.dae</uri>
                         <scale>1 1 1</scale>
                     </mesh>
@@ -108,104 +194,4 @@
             </collision>
         </link>
-        <link name='${model_name}_Rotation'>
-            <inertial>
-                <mass>0.59</mass>
-                <inertia>
-                    <ixx>0.0006558</ixx>
-                    <ixy>0</ixy>
-                    <ixz>0</ixz>
-                    <iyy>0.00065583</iyy>
-                    <iyz>0</iyz>
-                    <izz>0.00074316</izz>
-                </inertia>
-                <pose>0 0 0 0 -0 0</pose>
-            </inertial>
-            <pose>${x + 6.9e-05} ${y} ${z + 0.026037} ${roll} ${pitch} ${yaw}</pose>
-            <gravity>1</gravity>
-            <self_collide>0</self_collide>
-            <kinematic>0</kinematic>
-            <enable_wind>0</enable_wind>
-            <visual name='visual'>
-                <pose>0 0 0 0 -0 0</pose>
-                <geometry>
-                    <mesh>
-                        <uri>$(find robot_simulation)/models/SDS_Module/SDS_Rotation.dae</uri>
-                        <scale>1 1 1</scale>
-                    </mesh>
-                </geometry>
-                <material>
-                    <lighting>1</lighting>
-                    <script>
-                        <uri>file://media/materials/scripts/gazebo.material</uri>
-                        <name>Gazebo/Grey</name>
-                    </script>
-                    <shader type='pixel'>
-                        <normal_map>__default__</normal_map>
-                    </shader>
-                    <ambient>0.3 0.3 0.3 1</ambient>
-                    <diffuse>0.7 0.7 0.7 1</diffuse>
-                    <specular>0.01 0.01 0.01 1</specular>
-                    <emissive>0 0 0 1</emissive>
-                </material>
-                <transparency>0</transparency>
-                <cast_shadows>1</cast_shadows>
-            </visual>
-            <collision name='collision'>
-                <laser_retro>0</laser_retro>
-                <max_contacts>10</max_contacts>
-                <pose>0 0 0 0 -0 0</pose>
-                <geometry>
-                    <mesh>
-                        <uri>$(find robot_simulation)/models/SDS_Module/SDS_Rotation_Collision.dae</uri>
-                        <scale>1 1 1</scale>
-                    </mesh>
-                </geometry>
-                <surface>
-                    <friction>
-                        <ode>
-                            <mu>1</mu>
-                            <mu2>1</mu2>
-                            <fdir1>0 0 0</fdir1>
-                            <slip1>0</slip1>
-                            <slip2>0</slip2>
-                        </ode>
-                        <torsional>
-                            <coefficient>1</coefficient>
-                            <patch_radius>0</patch_radius>
-                            <surface_radius>0</surface_radius>
-                            <use_patch_radius>1</use_patch_radius>
-                            <ode>
-                                <slip>0</slip>
-                            </ode>
-                        </torsional>
-                    </friction>
-                    <bounce>
-                        <restitution_coefficient>0</restitution_coefficient>
-                        <threshold>1e+06</threshold>
-                    </bounce>
-                    <contact>
-                        <collide_without_contact>0</collide_without_contact>
-                        <collide_without_contact_bitmask>1</collide_without_contact_bitmask>
-                        <collide_bitmask>1</collide_bitmask>
-                        <ode>
-                            <soft_cfm>0</soft_cfm>
-                            <soft_erp>0.2</soft_erp>
-                            <kp>1e+13</kp>
-                            <kd>1</kd>
-                            <max_vel>0.01</max_vel>
-                            <min_depth>0</min_depth>
-                        </ode>
-                        <bullet>
-                            <split_impulse>1</split_impulse>
-                            <split_impulse_penetration_threshold>-0.01</split_impulse_penetration_threshold>
-                            <soft_cfm>0</soft_cfm>
-                            <soft_erp>0.2</soft_erp>
-                            <kp>1e+13</kp>
-                            <kd>1</kd>
-                        </bullet>
-                    </contact>
-                </surface>
-            </collision>
-        </link>
         <link name='${model_name}_Wheel'>
             <inertial>
@@ -234,18 +220,4 @@
                     </mesh>
                 </geometry>
-                <material>
-                    <lighting>1</lighting>
-                    <script>
-                        <uri>file://media/materials/scripts/gazebo.material</uri>
-                        <name>Gazebo/Grey</name>
-                    </script>
-                    <shader type='pixel'>
-                        <normal_map>__default__</normal_map>
-                    </shader>
-                    <ambient>0.3 0.3 0.3 1</ambient>
-                    <diffuse>0.7 0.7 0.7 1</diffuse>
-                    <specular>0.01 0.01 0.01 1</specular>
-                    <emissive>0 0 0 1</emissive>
-                </material>
                 <transparency>0</transparency>
                 <cast_shadows>1</cast_shadows>

Commit message: Testing

File: src/robot_simulation/models/SDS_Chassis/model.xacro (robot description, xacro)
@@ -3,4 +3,5 @@
     <xacro:include filename="$(find robot_simulation)/models/SDS_Module/SDS_Module.xacro"/>
     <model name="SDS_Chassis">
+        <pose>0 0 0.068978 0 0 0</pose>
         <static>0</static>
         <allow_auto_disable>1</allow_auto_disable>
@@ -98,7 +99,7 @@
           </link>
           <xacro:SDL_Module suffix="FL" x="0.289486"    y="0.289486"    z="0.016516" parent_link="Frames" roll="0" pitch="0" yaw="0"/>
-          <xacro:SDL_Module suffix="FR" x="0.289486"    y="-0.289486"   z="0.016516" parent_link="Frames" roll="0" pitch="0" yaw="-1.5708"/>
-          <xacro:SDL_Module suffix="BL" x="-0.289486"   y="0.289486"    z="0.016516" parent_link="Frames" roll="0" pitch="0" yaw="1.5708"/>
-          <xacro:SDL_Module suffix="BR" x="-0.289486"   y="-0.289486"   z="0.016516" parent_link="Frames" roll="0" pitch="0" yaw="-3.141516"/>
+          <xacro:SDL_Module suffix="FR" x="0.289486"    y="-0.289486"   z="0.016516" parent_link="Frames" roll="0" pitch="0" yaw="-1.5708"      rotation_offset="${1.5708}"/>
+          <xacro:SDL_Module suffix="BL" x="-0.289486"   y="0.289486"    z="0.016516" parent_link="Frames" roll="0" pitch="0" yaw="1.5708"       rotation_offset="${-1.5708}"/>
+          <xacro:SDL_Module suffix="BR" x="-0.289486"   y="-0.289486"   z="0.016516" parent_link="Frames" roll="0" pitch="0" yaw="-3.141516"    rotation_offset="${3.141516}"/>
     </model>
 </sdf>

File: src/robot_simulation/models/SDS_Module/SDS_Module.xacro (robot description, xacro)
@@ -1,5 +1,5 @@
 <?xml version='1.0'?>
 <sdf version='1.7' xmlns:xacro="http://www.ros.org/wiki/xacro">
-    <xacro:macro name="SDL_Module" params="suffix:='' parent_link:='' x:=0 y:=0 z:=0 roll:=0 pitch:=0 yaw:=0">
+    <xacro:macro name="SDL_Module" params="suffix:='' parent_link:='' x:=0 y:=0 z:=0 roll:=0 pitch:=0 yaw:=0 rotation_offset:=0">
         <xacro:if value="${suffix == ''}">
             <xacro:property name="model_name" value="SDS_Module" />
@@ -107,5 +107,5 @@
                 <pose>0 0 0 0 -0 0</pose>
             </inertial>
-            <pose>${x + 6.9e-05} ${y} ${z + 0.026037} ${roll} ${pitch} ${yaw}</pose>
+            <pose>${x + 6.9e-05} ${y} ${z + 0.026037} ${roll} ${pitch} ${yaw + rotation_offset}</pose>
             <gravity>1</gravity>
             <self_collide>0</self_collide>
@@ -120,18 +120,4 @@
                     </mesh>
                 </geometry>
-                <material>
-                    <lighting>1</lighting>
-                    <script>
-                        <uri>file://media/materials/scripts/gazebo.material</uri>
-                        <name>Gazebo/Grey</name>
-                    </script>
-                    <shader type='pixel'>
-                        <normal_map>__default__</normal_map>
-                    </shader>
-                    <ambient>0.3 0.3 0.3 1</ambient>
-                    <diffuse>0.7 0.7 0.7 1</diffuse>
-                    <specular>0.01 0.01 0.01 1</specular>
-                    <emissive>0 0 0 1</emissive>
-                </material>
                 <transparency>0</transparency>
                 <cast_shadows>1</cast_shadows>
@@ -207,5 +193,5 @@
                 <pose>0 0 0 0 -0 0</pose>
             </inertial>
-            <pose>${x -0.000137} ${y} ${z -0.034957} ${roll} ${pitch} ${yaw}</pose>
+            <pose>${x -0.000137} ${y} ${z -0.034957} ${roll} ${pitch} ${yaw + rotation_offset}</pose>
             <gravity>1</gravity>
             <self_collide>0</self_collide>
@@ -236,44 +222,14 @@
                     <friction>
                         <ode>
-                            <mu>1</mu>
-                            <mu2>1</mu2>
-                            <fdir1>0 0 0</fdir1>
-                            <slip1>0</slip1>
-                            <slip2>0</slip2>
-                        </ode>
-                        <torsional>
-                            <coefficient>1</coefficient>
-                            <patch_radius>0</patch_radius>
-                            <surface_radius>0</surface_radius>
-                            <use_patch_radius>1</use_patch_radius>
-                            <ode>
-                                <slip>0</slip>
-                            </ode>
-                        </torsional>
+                            <mu>1.16</mu>
+                            <mu2>1.16</mu2>
+                        </ode>
                     </friction>
-                    <bounce>
-                        <restitution_coefficient>0</restitution_coefficient>
-                        <threshold>1e+06</threshold>
-                    </bounce>
                     <contact>
-                        <collide_without_contact>0</collide_without_contact>
-                        <collide_without_contact_bitmask>1</collide_without_contact_bitmask>
-                        <collide_bitmask>1</collide_bitmask>
-                        <ode>
-                            <soft_cfm>0</soft_cfm>
-                            <soft_erp>0.2</soft_erp>
-                            <kp>1e+13</kp>
-                            <kd>1</kd>
-                            <max_vel>0.01</max_vel>
-                            <min_depth>0</min_depth>
-                        </ode>
-                        <bullet>
-                            <split_impulse>1</split_impulse>
-                            <split_impulse_penetration_threshold>-0.01</split_impulse_penetration_threshold>
-                            <soft_cfm>0</soft_cfm>
-                            <soft_erp>0.2</soft_erp>
-                            <kp>1e+13</kp>
-                            <kd>1</kd>
-                        </bullet>
+                        <ode>
+                            <min_depth>0.01</min_depth>
+                            <kp>1e15</kp>
+                            <kd>1e13</kd>
+                        </ode>
                     </contact>
                 </surface>
@@ -283,5 +239,4 @@
             <parent>${model_name}_Fixed</parent>
             <child>${model_name}_Rotation</child>
-            <pose>0 0 0 0 -0 0</pose>
             <axis>
                 <xyz>0 0 1</xyz>
@@ -295,6 +250,6 @@
                     <spring_reference>0</spring_reference>
                     <spring_stiffness>0</spring_stiffness>
-                    <damping>0.17</damping>
-                    <friction>0.0</friction>
+                    <damping>0.02</damping>
+                    <friction>3.5</friction>
                 </dynamics>
             </axis>
@@ -327,5 +282,5 @@
                     <spring_reference>0</spring_reference>
                     <spring_stiffness>0</spring_stiffness>
-                    <damping>0.04</damping>
+                    <damping>0.01</damping>
                     <friction>0.0</friction>
                 </dynamics>
@@ -355,4 +310,5 @@
             <torque_axis>z</torque_axis>
             <motor_model>Falcon</motor_model>
+            <inverted>true</inverted>
             <gear_ratio>21.4285714286</gear_ratio>
         </plugin>
