Commit message: FRC 2024 field and FirstCAD7421 reductions tuned

File: src/robot_simulation/models/FRC_Field_2024/model.xacro (robot description, xacro)
@@ -1,49 +1,8 @@
 <?xml version='1.0'?>
 <sdf version='1.7' xmlns:xacro="http://www.ros.org/wiki/xacro">
-    <model name='ground_plane'>
+    <xacro:include filename="$(find robot_simulation)/models/FRC_Field_2024/FRC_Field_2024.xacro"/>
+    <model name="FRC_Field_2024">
         <static>1</static>
-        <link name='link'>
-            <collision name='collision'>
-                <geometry>
-                    <mesh>
-                        <uri>$(find robot_simulation)/models/FRC_Field_2024/FRC_Field_2024_Collision.dae</uri>
-                        <scale>1 1 1</scale>
-                    </mesh>
-                </geometry>
-                <surface>
-                    <contact>
-                        <collide_bitmask>65535</collide_bitmask>
-                        <ode>
-                            <min_depth>0.01</min_depth>
-                            <kp>1e15</kp>
-                            <kd>1e13</kd>
-                        </ode>
-                    </contact>
-                    <friction>
-                        <ode>
-                            <mu>100</mu>
-                            <mu2>100</mu2>
-                        </ode>
-                        <torsional>
-                            <ode/>
-                        </torsional>
-                    </friction>
-                    <bounce/>
-                </surface>
-                <max_contacts>10</max_contacts>
-            </collision>
-            <visual name='visual'>
-                <cast_shadows>0</cast_shadows>
-                <geometry>
-                    <mesh>
-                        <uri>$(find robot_simulation)/models/FRC_Field_2024/FRC_Field_2024.dae</uri>
-                        <scale>1 1 1</scale>
-                    </mesh>
-                </geometry>
-            </visual>
-            <self_collide>0</self_collide>
-            <enable_wind>0</enable_wind>
-            <kinematic>0</kinematic>
-        </link>
+        <xacro:FRC_Field_2024/>
     </model>
 </sdf>

File: src/robot_simulation/models/FirstCAD7421/model.xacro (robot description, xacro)
@@ -884,5 +884,5 @@
             <torque_axis>y</torque_axis>
             <motor_model>FalconFOC</motor_model>
-            <gear_ratio>251</gear_ratio>
+            <gear_ratio>230</gear_ratio>
             <suffix>right</suffix>
         </plugin>
@@ -892,5 +892,5 @@
             <torque_axis>y</torque_axis>
             <motor_model>FalconFOC</motor_model>
-            <gear_ratio>251</gear_ratio>
+            <gear_ratio>230</gear_ratio>
             <suffix>left</suffix>
             <mechanically_inverted>true</mechanically_inverted>
@@ -901,5 +901,5 @@
             <torque_axis>y</torque_axis>
             <motor_model>FalconFOC</motor_model>
-            <gear_ratio>150</gear_ratio>
+            <gear_ratio>90</gear_ratio>
         </plugin>
         <plugin name='NTMotor_FirstCAD7421_Intake' filename='libnt_motor_plugin.so'>
@@ -938,5 +938,5 @@
             <torque_axis>y</torque_axis>
             <motor_model>FalconFOC</motor_model>
-            <gear_ratio>150</gear_ratio>
+            <gear_ratio>106</gear_ratio>
         </plugin>
         <plugin name='NTMotor_FirstCAD7421_Arm_Encoder' filename='libnt_cancoder_plugin.so'>
