Commit message: Testing pathplanner, fixed collision meshes with Meshlab

File: src/robot_simulation/models/FRC_Field_2024/FRC_Field_2024.xacro (robot description, xacro)
@@ -20,26 +20,4 @@
                 <max_contacts>10</max_contacts>
                 <surface>
-                    <friction>
-                        <ode>
-                            <mu>1</mu>
-                            <mu2>1</mu2>
-                            <fdir1>0 0 0</fdir1>
-                            <slip1>0</slip1>
-                            <slip2>0</slip2>
-                        </ode>
-                        <torsional>
-                            <coefficient>1</coefficient>
-                            <patch_radius>0</patch_radius>
-                            <surface_radius>0</surface_radius>
-                            <use_patch_radius>1</use_patch_radius>
-                            <ode>
-                                <slip>0</slip>
-                            </ode>
-                        </torsional>
-                    </friction>
-                    <bounce>
-                        <restitution_coefficient>0</restitution_coefficient>
-                        <threshold>1e+05</threshold>
-                    </bounce>
                     <contact>
                         <collide_without_contact>0</collide_without_contact>
@@ -49,5 +27,5 @@
                             <soft_cfm>0</soft_cfm>
                             <soft_erp>0.2</soft_erp>
-                            <kp>1e+13</kp>
+                            <kp>100000</kp>
                             <kd>1</kd>
                             <max_vel>0.001</max_vel>

File: src/robot_simulation/models/FirstCAD7421/model.xacro (robot description, xacro)
@@ -220,5 +220,5 @@
                 <pose>0 0 0 0 -0 0</pose>
             </inertial>
-            <pose>0.317256 0.254208 0.579382 1.5708 -0 0</pose>
+            <pose>0.317256 0.254208 0.569124 1.5708 -0 0</pose>
             <gravity>1</gravity>
             <self_collide>0</self_collide>
@@ -283,5 +283,5 @@
                 <pose>0 0 0 0 -0 0</pose>
             </inertial>
-            <pose>0.317256 -0.254208 0.579382 1.5708 -0 0</pose>
+            <pose>0.317256 -0.254208 0.569124 1.5708 -0 0</pose>
             <gravity>1</gravity>
             <self_collide>0</self_collide>
@@ -635,4 +635,5 @@
                     <spring_stiffness>0</spring_stiffness>
                     <damping>0.75</damping>
+                    <friction>0.02</friction>
                 </dynamics>
             </axis>
@@ -666,4 +667,5 @@
                     <spring_stiffness>0</spring_stiffness>
                     <damping>0.1</damping>
+                    <friction>0.02</friction>
                 </dynamics>
             </axis>
@@ -760,6 +762,6 @@
                     <spring_reference>0</spring_reference>
                     <spring_stiffness>0</spring_stiffness>
-                    <damping>0.001</damping>
-                    <friction>0.005</friction>
+                    <damping>0.02</damping>
+                    <friction>0.01</friction>
                 </dynamics>
             </axis>
@@ -792,6 +794,6 @@
                     <spring_reference>0</spring_reference>
                     <spring_stiffness>0</spring_stiffness>
-                    <damping>0.001</damping>
-                    <friction>0.005</friction>
+                    <damping>0.02</damping>
+                    <friction>0.01</friction>
                 </dynamics>
             </axis>

File: src/robot_simulation/models/SDS_Module/SDS_Module.xacro (robot description, xacro)
@@ -219,4 +219,19 @@
                     </mesh>
                 </geometry>
+                <surface>
+                    <friction>
+                        <ode>
+                            <mu>1.16</mu>
+                            <mu2>1.16</mu2>
+                        </ode>
+                    </friction>
+                    <contact>
+                        <ode>
+                            <min_depth>0.001</min_depth>
+                            <kp>1e15</kp>
+                            <kd>1</kd>
+                        </ode>
+                    </contact>
+                </surface>
             </collision>
         </link>
@@ -243,10 +258,6 @@
                     <limit>
                         <cfm>0</cfm>
-                        <erp>0.2</erp>
+                        <erp>0</erp>
                     </limit>
-                    <suspension>
-                        <cfm>0</cfm>
-                        <erp>0.2</erp>
-                    </suspension>
                 </ode>
             </physics>
@@ -265,22 +276,8 @@
                 </limit>
                 <dynamics>
-                    <spring_reference>0</spring_reference>
-                    <spring_stiffness>0</spring_stiffness>
-                    <damping>0.04</damping>
-                    <friction>0.02</friction>
+                    <damping>0.01</damping>
+                    <friction>0.01</friction>
                 </dynamics>
             </axis>
-            <physics>
-                <ode>
-                    <limit>
-                        <cfm>0.0</cfm>
-                        <erp>0.2</erp>
-                    </limit>
-                    <suspension>
-                        <cfm>0</cfm>
-                        <erp>0.2</erp>
-                    </suspension>
-                </ode>
-            </physics>
         </joint>
         <xacro:unless value="${parent_link == ''}">

File: src/robot_simulation/worlds/frc_2024.xacro (robot description, xacro)
@@ -60,5 +60,5 @@
                             <ode>
                                 <max_vel>0.001</max_vel>
-                                <min_depth>0</min_depth>
+                                <min_depth>0.001</min_depth>
                                 <kp>1e15</kp>
                                 <kd>1e13</kd>
@@ -94,5 +94,5 @@
                 <constraints>
                     <contact_max_correcting_vel>0.1</contact_max_correcting_vel>
-                    <contact_surface_layer>0.0001</contact_surface_layer>
+                    <contact_surface_layer>0.001</contact_surface_layer>
                 </constraints>
             </ode>
@@ -120,12 +120,6 @@
             <iterations>14042</iterations>
             <model name='FRC_Field_2024'>
-                <pose>0 0 -0.005000 0 -0 0</pose>
+                <pose>0 0 -0.005000 0 -0 3.141516</pose>
                 <scale>1 1 1</scale>
-                <link name='field'>
-                    <pose>0 0 0 0 -0 0</pose>
-                    <velocity>0 0 0 0 -0 0</velocity>
-                    <acceleration>0 0 0 0 -0 0</acceleration>
-                    <wrench>0 0 0 0 -0 0</wrench>
-                </link>
             </model>
         </state>

Commit message: Fine tuning

File: src/robot_simulation/models/FRC_Field_2024/FRC_Field_2024.xacro (robot description, xacro)
@@ -21,16 +21,22 @@
                 <surface>
                     <contact>
-                        <collide_without_contact>0</collide_without_contact>
-                        <collide_without_contact_bitmask>1</collide_without_contact_bitmask>
-                        <collide_bitmask>1</collide_bitmask>
+                        <collide_bitmask>65535</collide_bitmask>
                         <ode>
-                            <soft_cfm>0</soft_cfm>
-                            <soft_erp>0.2</soft_erp>
-                            <kp>100000</kp>
-                            <kd>1</kd>
                             <max_vel>0.001</max_vel>
-                            <min_depth>0</min_depth>
+                            <min_depth>0.001</min_depth>
+                            <kp>1e15</kp>
+                            <kd>1e13</kd>
                         </ode>
                     </contact>
+                    <friction>
+                        <ode>
+                            <mu>100</mu>
+                            <mu2>100</mu2>
+                        </ode>
+                        <torsional>
+                            <ode/>
+                        </torsional>
+                    </friction>
+                    <bounce/>
                 </surface>
             </collision>

File: src/robot_simulation/models/SDS_Module/SDS_Module.xacro (robot description, xacro)
@@ -50,45 +50,11 @@
                     <friction>
                         <ode>
-                            <mu>1</mu>
-                            <mu2>1</mu2>
+                            <mu>0.9</mu>
+                            <mu2>0.9</mu2>
                             <fdir1>0 0 0</fdir1>
                             <slip1>0</slip1>
                             <slip2>0</slip2>
                         </ode>
-                        <torsional>
-                            <coefficient>1</coefficient>
-                            <patch_radius>0</patch_radius>
-                            <surface_radius>0</surface_radius>
-                            <use_patch_radius>1</use_patch_radius>
-                            <ode>
-                                <slip>0</slip>
-                            </ode>
-                        </torsional>
                     </friction>
-                    <bounce>
-                        <restitution_coefficient>0</restitution_coefficient>
-                        <threshold>1e+06</threshold>
-                    </bounce>
-                    <contact>
-                        <collide_without_contact>0</collide_without_contact>
-                        <collide_without_contact_bitmask>1</collide_without_contact_bitmask>
-                        <collide_bitmask>1</collide_bitmask>
-                        <ode>
-                            <soft_cfm>0</soft_cfm>
-                            <soft_erp>0.2</soft_erp>
-                            <kp>1e+13</kp>
-                            <kd>1</kd>
-                            <max_vel>0.01</max_vel>
-                            <min_depth>0</min_depth>
-                        </ode>
-                        <bullet>
-                            <split_impulse>1</split_impulse>
-                            <split_impulse_penetration_threshold>-0.01</split_impulse_penetration_threshold>
-                            <soft_cfm>0</soft_cfm>
-                            <soft_erp>0.2</soft_erp>
-                            <kp>1e+13</kp>
-                            <kd>1</kd>
-                        </bullet>
-                    </contact>
                 </surface>
             </collision>
@@ -220,16 +186,23 @@
                 </geometry>
                 <surface>
+                    <contact>
+                        <collide_bitmask>65535</collide_bitmask>
+                        <ode>
+                            <max_vel>0.001</max_vel>
+                            <min_depth>0.001</min_depth>
+                            <kp>1e15</kp>
+                            <kd>1e13</kd>
+                        </ode>
+                    </contact>
                     <friction>
                         <ode>
-                            <mu>1.16</mu>
-                            <mu2>1.16</mu2>
-                        </ode>
+                            <mu>100</mu>
+                            <mu2>100</mu2>
+                        </ode>
+                        <torsional>
+                            <ode/>
+                        </torsional>
                     </friction>
-                    <contact>
-                        <ode>
-                            <kp>1e15</kp>
-                            <kd>1</kd>
-                        </ode>
-                    </contact>
+                    <bounce/>
                 </surface>
             </collision>
@@ -257,5 +230,5 @@
                     <limit>
                         <cfm>0</cfm>
-                        <erp>0</erp>
+                        <erp>0.8</erp>
                     </limit>
                 </ode>
@@ -276,7 +249,15 @@
                 <dynamics>
                     <damping>0.001</damping>
-                    <friction>0.1</friction>
+                    <friction>0.001</friction>
                 </dynamics>
             </axis>
+            <physics>
+                <ode>
+                    <limit>
+                        <cfm>0</cfm>
+                        <erp>0.8</erp>
+                    </limit>
+                </ode>
+            </physics>
         </joint>
         <xacro:unless value="${parent_link == ''}">

File: src/robot_simulation/worlds/frc_2024.xacro (robot description, xacro)
@@ -87,4 +87,6 @@
         <atmosphere type='adiabatic'/>
         <physics type='ode'>
+            <max_step_size>0.00050</max_step_size>
+            <real_time_update_rate>2000</real_time_update_rate>
             <ode>
                 <solver>
