Commit message: Added camera to FirstCAD7421

File: src/robot_simulation/models/FirstCAD7421/model.xacro (robot description, xacro)
@@ -2,5 +2,5 @@
 <sdf version='1.7' xmlns:xacro="http://www.ros.org/wiki/xacro">
     <xacro:include filename="$(find robot_simulation)/models/SDS_Module/SDS_Module.xacro"/>
-    <model name="7421-24">
+    <model name="FirstCAD7421">
         <pose>0 0 0.040368 0 0 0</pose>
         <static>0</static>
@@ -28,5 +28,5 @@
                 <geometry>
                     <mesh>
-                        <uri>$(find robot_simulation)/models/7421-24/Chassis.dae</uri>
+                        <uri>$(find robot_simulation)/models/FirstCAD7421/Chassis.dae</uri>
                         <scale>1 1 1</scale>
                     </mesh>
@@ -41,5 +41,5 @@
                 <geometry>
                     <mesh>
-                        <uri>$(find robot_simulation)/models/7421-24/Chassis_Collision.dae</uri>
+                        <uri>$(find robot_simulation)/models/FirstCAD7421/Chassis_Collision.dae</uri>
                         <scale>1 1 1</scale>
                     </mesh>
@@ -99,5 +99,5 @@
                 <geometry>
                     <mesh>
-                        <uri>$(find robot_simulation)/models/7421-24/Arm.dae</uri>
+                        <uri>$(find robot_simulation)/models/FirstCAD7421/Arm.dae</uri>
                         <scale>1 1 1</scale>
                     </mesh>
@@ -112,5 +112,5 @@
                 <geometry>
                     <mesh>
-                        <uri>$(find robot_simulation)/models/7421-24/Arm_Collision.dae</uri>
+                        <uri>$(find robot_simulation)/models/FirstCAD7421/Arm_Collision.dae</uri>
                         <scale>1 1 1</scale>
                     </mesh>
@@ -164,5 +164,5 @@
                 <geometry>
                     <mesh>
-                        <uri>$(find robot_simulation)/models/7421-24/Shooter.dae</uri>
+                        <uri>$(find robot_simulation)/models/FirstCAD7421/Shooter.dae</uri>
                         <scale>1 1 1</scale>
                     </mesh>
@@ -177,5 +177,5 @@
                 <geometry>
                     <mesh>
-                        <uri>$(find robot_simulation)/models/7421-24/Shooter_Collision.dae</uri>
+                        <uri>$(find robot_simulation)/models/FirstCAD7421/Shooter_Collision.dae</uri>
                         <scale>1 1 1</scale>
                     </mesh>
@@ -229,5 +229,5 @@
                 <geometry>
                     <mesh>
-                        <uri>$(find robot_simulation)/models/7421-24/StorageWheels.dae</uri>
+                        <uri>$(find robot_simulation)/models/FirstCAD7421/StorageWheels.dae</uri>
                     </mesh>
                 </geometry>
@@ -241,5 +241,5 @@
                 <geometry>
                     <mesh>
-                        <uri>$(find robot_simulation)/models/7421-24/StorageWheels_Collision.dae</uri>
+                        <uri>$(find robot_simulation)/models/FirstCAD7421/StorageWheels_Collision.dae</uri>
                     </mesh>
                 </geometry>
@@ -292,5 +292,5 @@
                 <geometry>
                     <mesh>
-                        <uri>$(find robot_simulation)/models/7421-24/StorageWheels.dae</uri>
+                        <uri>$(find robot_simulation)/models/FirstCAD7421/StorageWheels.dae</uri>
                     </mesh>
                 </geometry>
@@ -304,5 +304,5 @@
                 <geometry>
                     <mesh>
-                        <uri>$(find robot_simulation)/models/7421-24/StorageWheels_Collision.dae</uri>
+                        <uri>$(find robot_simulation)/models/FirstCAD7421/StorageWheels_Collision.dae</uri>
                     </mesh>
                 </geometry>
@@ -355,5 +355,5 @@
                 <geometry>
                     <mesh>
-                        <uri>$(find robot_simulation)/models/7421-24/ShooterRoller.dae</uri>
+                        <uri>$(find robot_simulation)/models/FirstCAD7421/ShooterRoller.dae</uri>
                     </mesh>
                 </geometry>
@@ -367,5 +367,5 @@
                 <geometry>
                     <mesh>
-                        <uri>$(find robot_simulation)/models/7421-24/ShooterRoller.dae</uri>
+                        <uri>$(find robot_simulation)/models/FirstCAD7421/ShooterRoller.dae</uri>
                     </mesh>
                 </geometry>
@@ -418,5 +418,5 @@
                 <geometry>
                     <mesh>
-                        <uri>$(find robot_simulation)/models/7421-24/ShooterRoller.dae</uri>
+                        <uri>$(find robot_simulation)/models/FirstCAD7421/ShooterRoller.dae</uri>
                     </mesh>
                 </geometry>
@@ -430,5 +430,5 @@
                 <geometry>
                     <mesh>
-                        <uri>$(find robot_simulation)/models/7421-24/ShooterRoller.dae</uri>
+                        <uri>$(find robot_simulation)/models/FirstCAD7421/ShooterRoller.dae</uri>
                         <scale>1 1 1</scale>
                     </mesh>
@@ -482,5 +482,5 @@
                 <geometry>
                     <mesh>
-                        <uri>$(find robot_simulation)/models/7421-24/Supports.dae</uri>
+                        <uri>$(find robot_simulation)/models/FirstCAD7421/Supports.dae</uri>
                     </mesh>
                 </geometry>
@@ -494,5 +494,5 @@
                 <geometry>
                     <mesh>
-                        <uri>$(find robot_simulation)/models/7421-24/Supports_Collision.dae</uri>
+                        <uri>$(find robot_simulation)/models/FirstCAD7421/Supports_Collision.dae</uri>
                     </mesh>
                 </geometry>
@@ -545,5 +545,5 @@
                 <geometry>
                     <mesh>
-                        <uri>$(find robot_simulation)/models/7421-24/IntakeWheels.dae</uri>
+                        <uri>$(find robot_simulation)/models/FirstCAD7421/IntakeWheels.dae</uri>
                     </mesh>
                 </geometry>
@@ -557,5 +557,5 @@
                 <geometry>
                     <mesh>
-                        <uri>$(find robot_simulation)/models/7421-24/IntakeWheels_Collision.dae</uri>
+                        <uri>$(find robot_simulation)/models/FirstCAD7421/IntakeWheels_Collision.dae</uri>
                     </mesh>
                 </geometry>
@@ -586,4 +586,47 @@
             </collision>
         </link>
+        <model name='camera'>
+            <static>true</static>
+            <pose>0.5 0 0.5 0 0 0</pose>
+            <link name='link'>
+                <visual name='visual'>
+                    <geometry>
+                        <box>
+                            <size>0.1 0.1 0.1</size>
+                        </box>
+                    </geometry>
+                </visual>
+                <sensor name='my_camera' type='camera'>
+                    <camera>
+                        <horizontal_fov>1.047</horizontal_fov>
+                        <image>
+                            <width>1920</width>
+                            <height>1080</height>
+                        </image>
+                        <clip>
+                            <near>0.1</near>
+                            <far>100</far>
+                        </clip>
+                    </camera>
+                    <always_on>1</always_on>
+                    <update_rate>120</update_rate>
+                    <plugin name="camera_controller" filename="libgazebo_ros_camera.so">
+                        <alwaysOn>true</alwaysOn>
+                        <updateRate>0.0</updateRate>
+                        <cameraName>camera</cameraName>
+                        <imageTopicName>image_raw</imageTopicName>
+                        <cameraInfoTopicName>camera_info</cameraInfoTopicName>
+                        <frameName>link</frameName>
+                        <robotNamespace>FirstCAD7421</robotNamespace>
+                        <hackBaseline>0.07</hackBaseline>
+                        <distortionK1>0.0</distortionK1>
+                        <distortionK2>0.0</distortionK2>
+                        <distortionK3>0.0</distortionK3>
+                        <distortionT1>0.0</distortionT1>
+                        <distortionT2>0.0</distortionT2>
+                    </plugin>
+                </sensor>
+            </link>
+        </model>
         <joint name='chassis_arm_joint' type='revolute'>
             <parent>chassis</parent>
@@ -839,5 +882,5 @@
             </physics>
         </joint>
-        <plugin name='NTMotor_7421-24_Arm_Right' filename='libnt_motor_plugin.so'>
+        <plugin name='NTMotor_FirstCAD7421_Arm_Right' filename='libnt_motor_plugin.so'>
             <joint_name>chassis_arm_joint</joint_name>
             <joint_axis>0</joint_axis>
@@ -847,5 +890,5 @@
             <suffix>right</suffix>
         </plugin>
-        <plugin name='NTMotor_7421-24_Arm_Left' filename='libnt_motor_plugin.so'>
+        <plugin name='NTMotor_FirstCAD7421_Arm_Left' filename='libnt_motor_plugin.so'>
             <joint_name>chassis_arm_joint</joint_name>
             <joint_axis>0</joint_axis>
@@ -856,5 +899,5 @@
             <mechanically_inverted>true</mechanically_inverted>
         </plugin>
-        <plugin name='NTMotor_7421-24_Shooter_Arm' filename='libnt_motor_plugin.so'>
+        <plugin name='NTMotor_FirstCAD7421_Shooter_Arm' filename='libnt_motor_plugin.so'>
             <joint_name>arm_shooter_joint</joint_name>
             <joint_axis>0</joint_axis>
@@ -863,5 +906,5 @@
             <gear_ratio>150</gear_ratio>
         </plugin>
-        <plugin name='NTMotor_7421-24_Intake' filename='libnt_motor_plugin.so'>
+        <plugin name='NTMotor_FirstCAD7421_Intake' filename='libnt_motor_plugin.so'>
             <joint_name>chassis_intake_wheels_joint</joint_name>
             <joint_axis>0</joint_axis>
@@ -870,5 +913,5 @@
             <gear_ratio>1</gear_ratio>
         </plugin>
-        <plugin name='NTMotor_7421-24_Shooter_Up' filename='libnt_motor_plugin.so'>
+        <plugin name='NTMotor_FirstCAD7421_Shooter_Up' filename='libnt_motor_plugin.so'>
             <joint_name>shooter_roller_up_joint</joint_name>
             <joint_axis>0</joint_axis>
@@ -877,5 +920,5 @@
             <gear_ratio>0.416666667</gear_ratio>
         </plugin>
-        <plugin name='NTMotor_7421-24_Shooter_Down' filename='libnt_motor_plugin.so'>
+        <plugin name='NTMotor_FirstCAD7421_Shooter_Down' filename='libnt_motor_plugin.so'>
             <joint_name>shooter_roller_down_joint</joint_name>
             <joint_axis>0</joint_axis>
@@ -885,5 +928,5 @@
             <mechanically_inverted>true</mechanically_inverted>
         </plugin>
-        <plugin name='NTMotor_7421-24_Storage' filename='libnt_motor_plugin.so'>
+        <plugin name='NTMotor_FirstCAD7421_Storage' filename='libnt_motor_plugin.so'>
             <joint_name>shooter_storage_wheel_left_joint</joint_name>
             <joint_axis>0</joint_axis>
@@ -893,5 +936,5 @@
             <mechanically_inverted>true</mechanically_inverted>
         </plugin>
-        <plugin name='NTMotor_7421-24_Supports' filename='libnt_motor_plugin.so'>
+        <plugin name='NTMotor_FirstCAD7421_Supports' filename='libnt_motor_plugin.so'>
             <joint_name>chassis_supports_joint</joint_name>
             <joint_axis>0</joint_axis>
@@ -900,17 +943,17 @@
             <gear_ratio>150</gear_ratio>
         </plugin>
-        <plugin name='NTMotor_7421-24_Arm_Encoder' filename='libnt_cancoder_plugin.so'>
+        <plugin name='NTMotor_FirstCAD7421_Arm_Encoder' filename='libnt_cancoder_plugin.so'>
             <joint_name>chassis_arm_joint</joint_name>
             <inverted>true</inverted>
         </plugin>
-        <plugin name='NTMotor_7421-24_Arm_Shooter_Encoder' filename='libnt_cancoder_plugin.so'>
+        <plugin name='NTMotor_FirstCAD7421_Arm_Shooter_Encoder' filename='libnt_cancoder_plugin.so'>
             <joint_name>arm_shooter_joint</joint_name>
             <inverted>true</inverted>
         </plugin>
-        <plugin name='NTMotor_7421-24_Support_Encoder' filename='libnt_cancoder_plugin.so'>
+        <plugin name='NTMotor_FirstCAD7421_Support_Encoder' filename='libnt_cancoder_plugin.so'>
             <joint_name>chassis_supports_joint</joint_name>
             <inverted>true</inverted>
         </plugin>
-        <plugin name='LinkedJoint_7421-24_Storage_Wheels' filename='liblinked_joint_plugin.so'>
+        <plugin name='LinkedJoint_FirstCAD7421_Storage_Wheels' filename='liblinked_joint_plugin.so'>
             <motor_name>shooter_storage_wheel_left_joint</motor_name>
             <joint_target_name>shooter_storage_wheel_right_joint</joint_target_name>

Commit message: Implement cameras, stream them to http so PhotonVision can read them

File: src/robot_simulation/models/FirstCAD7421/model.xacro (robot description, xacro)
@@ -586,43 +586,40 @@
             </collision>
         </link>
-        <model name='camera'>
-            <static>true</static>
+        <link name='test_camera'>
             <pose>0.5 0 0.5 0 0 0</pose>
-            <link name='link'>
-                <visual name='visual'>
-                    <geometry>
-                        <box>
-                            <size>0.1 0.1 0.1</size>
-                        </box>
-                    </geometry>
-                </visual>
-                <sensor name='my_camera' type='camera'>
-                    <camera>
-                        <horizontal_fov>1.047</horizontal_fov>
-                        <image>
-                            <width>1920</width>
-                            <height>1080</height>
-                        </image>
-                    </camera>
-                    <always_on>1</always_on>
-                    <update_rate>120</update_rate>
-                    <plugin name="camera_controller" filename="libgazebo_ros_camera.so">
-                        <alwaysOn>true</alwaysOn>
-                        <updateRate>120</updateRate>
-                        <cameraName>camera</cameraName>
-                        <imageTopicName>image_raw</imageTopicName>
-                        <cameraInfoTopicName>camera_info</cameraInfoTopicName>
-                        <frameName>link</frameName>
-                        <robotNamespace>FirstCAD7421</robotNamespace>
-                        <hackBaseline>0.07</hackBaseline>
-                        <distortionK1>0.0</distortionK1>
-                        <distortionK2>0.0</distortionK2>
-                        <distortionK3>0.0</distortionK3>
-                        <distortionT1>0.0</distortionT1>
-                        <distortionT2>0.0</distortionT2>
-                    </plugin>
-                </sensor>
-            </link>
-        </model>
+            <visual name='visual'>
+                <geometry>
+                    <box>
+                        <size>0.1 0.1 0.1</size>
+                    </box>
+                </geometry>
+            </visual>
+            <sensor name='my_camera' type='camera'>
+                <camera>
+                    <horizontal_fov>1.047</horizontal_fov>
+                    <image>
+                        <width>1920</width>
+                        <height>1080</height>
+                    </image>
+                </camera>
+                <always_on>1</always_on>
+                <update_rate>120</update_rate>
+                <plugin name="camera_controller" filename="libgazebo_ros_camera.so">
+                    <alwaysOn>true</alwaysOn>
+                    <updateRate>120</updateRate>
+                    <cameraName>camera</cameraName>
+                    <imageTopicName>image_raw</imageTopicName>
+                    <cameraInfoTopicName>camera_info</cameraInfoTopicName>
+                    <frameName>test_camera</frameName>
+                    <robotNamespace>FirstCAD7421</robotNamespace>
+                    <hackBaseline>0.07</hackBaseline>
+                    <distortionK1>0.0</distortionK1>
+                    <distortionK2>0.0</distortionK2>
+                    <distortionK3>0.0</distortionK3>
+                    <distortionT1>0.0</distortionT1>
+                    <distortionT2>0.0</distortionT2>
+                </plugin>
+            </sensor>
+        </link>
         <joint name='chassis_arm_joint' type='revolute'>
             <parent>chassis</parent>
@@ -878,4 +875,8 @@
             </physics>
         </joint>
+        <joint name='chassis_test_camera' type='fixed'>
+            <parent>chassis</parent>
+            <child>test_camera</child>
+        </joint>
         <plugin name='NTMotor_FirstCAD7421_Arm_Right' filename='libnt_motor_plugin.so'>
             <joint_name>chassis_arm_joint</joint_name>

File: src/robot_simulation/models/SDS_Module/SDS_Module.xacro (robot description, xacro)
@@ -228,5 +228,5 @@
                     <contact>
                         <ode>
-                            <min_depth>0.001</min_depth>
+                            <min_depth>0.01</min_depth>
                             <kp>1e15</kp>
                             <kd>1</kd>

Commit message: Update to NT4

File: src/robot_simulation/models/FirstCAD7421/model.xacro (robot description, xacro)
@@ -335,10 +335,10 @@
         <link name='shooter_roller_up'>
             <inertial>
-                <mass>0.680389</mass>
+                <mass>0.2</mass>
                 <inertia>
-                    <ixx>0.00631</ixx>
+                    <ixx>0.03211556</ixx>
                     <ixy>0</ixy>
                     <ixz>0</ixz>
-                    <iyy>0.03211556</iyy>
+                    <iyy>0.000631</iyy>
                     <iyz>0</iyz>
                     <izz>0.01211556</izz>
@@ -398,10 +398,10 @@
         <link name='shooter_roller_down'>
             <inertial>
-                <mass>0.680389</mass>
+                <mass>0.2</mass>
                 <inertia>
-                    <ixx>0.00631</ixx>
+                    <ixx>0.03211556</ixx>
                     <ixy>0</ixy>
                     <ixz>0</ixz>
-                    <iyy>0.03211556</iyy>
+                    <iyy>0.000631</iyy>
                     <iyz>0</iyz>
                     <izz>0.01211556</izz>
@@ -762,6 +762,6 @@
                     <spring_reference>0</spring_reference>
                     <spring_stiffness>0</spring_stiffness>
-                    <damping>0.02</damping>
-                    <friction>0.01</friction>
+                    <damping>0.001</damping>
+                    <friction>0.0</friction>
                 </dynamics>
             </axis>
@@ -794,6 +794,6 @@
                     <spring_reference>0</spring_reference>
                     <spring_stiffness>0</spring_stiffness>
-                    <damping>0.02</damping>
-                    <friction>0.01</friction>
+                    <damping>0.001</damping>
+                    <friction>0.0</friction>
                 </dynamics>
             </axis>
@@ -908,5 +908,5 @@
             <torque_axis>y</torque_axis>
             <motor_model>FalconFOC</motor_model>
-            <gear_ratio>1</gear_ratio>
+            <gear_ratio>3</gear_ratio>
         </plugin>
         <plugin name='NTMotor_FirstCAD7421_Shooter_Up' filename='libnt_motor_plugin.so'>
@@ -915,5 +915,5 @@
             <torque_axis>y</torque_axis>
             <motor_model>FalconFOC</motor_model>
-            <gear_ratio>0.416666667</gear_ratio>
+            <gear_ratio>3</gear_ratio>
         </plugin>
         <plugin name='NTMotor_FirstCAD7421_Shooter_Down' filename='libnt_motor_plugin.so'>
@@ -922,5 +922,5 @@
             <torque_axis>y</torque_axis>
             <motor_model>FalconFOC</motor_model>
-            <gear_ratio>0.416666667</gear_ratio>
+            <gear_ratio>3</gear_ratio>
             <mechanically_inverted>true</mechanically_inverted>
         </plugin>
@@ -930,5 +930,5 @@
             <torque_axis>y</torque_axis>
             <motor_model>FalconFOC</motor_model>
-            <gear_ratio>1</gear_ratio>
+            <gear_ratio>3</gear_ratio>
             <mechanically_inverted>true</mechanically_inverted>
         </plugin>
