Commit message: Add photonvision and driver cameras to Vantage model

File: src/robot_simulation/models/SDS_Module/SDS_Module.xacro (robot description, xacro)
@@ -277,5 +277,5 @@
                 <dynamics>
                     <damping>0.01</damping>
-                    <friction>0.01</friction>
+                    <friction>0.25</friction>
                 </dynamics>
             </axis>

File: src/robot_simulation/models/Vantage7421/model.xacro (robot description, xacro)
@@ -474,4 +474,70 @@
                 </surface>
             </collision>
+        </link>
+        <link name='photonvision_camera'>
+            <pose>-0.330107 0 0.312850 0 -0.4 3.141516</pose>
+            <visual name='visual'>
+                <geometry>
+                    <box>
+                        <size>0.01 0.01 0.01</size>
+                    </box>
+                </geometry>
+            </visual>
+            <sensor name='photonvision_sensor' type='camera'>
+                <camera>
+                    <horizontal_fov>1.22173</horizontal_fov>
+                    <image>
+                        <width>1280</width>
+                        <height>800</height>
+                    </image>
+                    <lens>
+                        <scale_to_fov>true</scale_to_fov>
+                    </lens>
+                </camera>
+                <always_on>1</always_on>
+                <update_rate>60</update_rate>
+                <plugin name="camera_controller" filename="libgazebo_ros_camera.so">
+                    <alwaysOn>true</alwaysOn>
+                    <updateRate>60</updateRate>
+                    <cameraName>photonvision</cameraName>
+                    <imageTopicName>image_raw</imageTopicName>
+                    <cameraInfoTopicName>camera_info</cameraInfoTopicName>
+                    <frameName>photonvision_camera</frameName>
+                    <robotNamespace>Vantage7421</robotNamespace>
+                </plugin>
+            </sensor>
+        </link>
+        <link name='driver_camera'>
+            <pose>0.276743 0 0.639094 0 -0.610865 0</pose>
+            <visual name='visual'>
+                <geometry>
+                    <box>
+                        <size>0.01 0.01 0.01</size>
+                    </box>
+                </geometry>
+            </visual>
+            <sensor name='driver_sensor' type='camera'>
+                <camera>
+                    <horizontal_fov>1.22173</horizontal_fov>
+                    <image>
+                        <width>640</width>
+                        <height>360</height>
+                    </image>
+                    <lens>
+                        <scale_to_fov>true</scale_to_fov>
+                    </lens>
+                </camera>
+                <always_on>1</always_on>
+                <update_rate>60</update_rate>
+                <plugin name="camera_controller" filename="libgazebo_ros_camera.so">
+                    <alwaysOn>true</alwaysOn>
+                    <updateRate>60</updateRate>
+                    <cameraName>driver</cameraName>
+                    <imageTopicName>image_raw</imageTopicName>
+                    <cameraInfoTopicName>camera_info</cameraInfoTopicName>
+                    <frameName>driver_camera</frameName>
+                    <robotNamespace>Vantage7421</robotNamespace>
+                </plugin>
+            </sensor>
         </link>
         <xacro:ShooterRoller suffix="up" x="0.002463" y="-0.006387" z="0.619108" roll="0" pitch="0" yaw="0"/>
@@ -802,4 +868,12 @@
             </physics>
         </joint>
+        <joint name='chassis_photonvision_camera' type='fixed'>
+            <parent>chassis</parent>
+            <child>photonvision_camera</child>
+        </joint>
+        <joint name='chassis_driver_camera' type='fixed'>
+            <parent>shooter</parent>
+            <child>driver_camera</child>
+        </joint>
         <plugin name='NTMotor_Vantage7421_Arm_Right' filename='libnt_motor_plugin.so'>
             <joint_name>chassis_arm_joint</joint_name>
